File: LM5032 Boost Converter Sch.kicad_pcb (KiCad board)
At the start: 2 copper layers, 48 parts, among them Q1 NMOS, Q10 NMOS, Q11 NMOS, Q12 NMOS, Q13 NMOS, Q14 NMOS, Q15 NMOS, Q16 NMOS, Q2 NMOS, Q3 NMOS, Q4 NMOS, Q5 NMOS, Q6 NMOS, Q7 NMOS, Q8 NMOS, Q9 NMOS

Commit message: update
Parts:
- removed REF** (x16): T220 Heatsink, Library:T220 Heatsink
- added C1: 1uF, Capacitor_SMD:C_1206_3216Metric_Pad1.33x1.80mm_HandSolder, F.Cu at (123.9, 207.8)
- added C100: 10uF, Capacitor_SMD:C_1210_3225Metric_Pad1.33x2.70mm_HandSolder, F.Cu at (133.2, 140.3)
- added C101: 100nF, Capacitor_SMD:C_1206_3216Metric_Pad1.33x1.80mm_HandSolder, F.Cu at (133.2, 144.4)
- added C102: 56nF, Capacitor_SMD:C_1206_3216Metric_Pad1.33x1.80mm_HandSolder, F.Cu at (124.0, 145.3)
- added C103: 2.2uF, Capacitor_SMD:C_1206_3216Metric_Pad1.33x1.80mm_HandSolder, F.Cu at (112.9, 149.6)
- added C104: 100nF, Capacitor_SMD:C_1206_3216Metric_Pad1.33x1.80mm_HandSolder, F.Cu at (121.7, 163.9)
- added C105: 100nF, Capacitor_SMD:C_1206_3216Metric_Pad1.33x1.80mm_HandSolder, F.Cu at (116.5, 157.5)
- added C106: 8.2nF, Capacitor_SMD:C_1206_3216Metric_Pad1.33x1.80mm_HandSolder, F.Cu at (125.5, 135.4)
- added C107: 470pF, Capacitor_SMD:C_1206_3216Metric_Pad1.33x1.80mm_HandSolder, F.Cu at (125.5, 139.1)
- added C108: 820pF, Capacitor_SMD:C_1206_3216Metric_Pad1.33x1.80mm_HandSolder, F.Cu at (118.2, 178.1)
- added C109: 22uF, Capacitor_SMD:C_1206_3216Metric_Pad1.33x1.80mm_HandSolder, F.Cu at (113.0, 184.2)
- added C2: 1uF, Capacitor_SMD:C_1206_3216Metric_Pad1.33x1.80mm_HandSolder, F.Cu at (130.7, 207.8)
- added C200: 470pF, Capacitor_SMD:C_1206_3216Metric_Pad1.33x1.80mm_HandSolder, F.Cu at (158.4, 162.1)
- added C201: 0.1uF, Capacitor_SMD:C_1206_3216Metric_Pad1.33x1.80mm_HandSolder, F.Cu at (164.2, 163.2)
- added C202: 0.1uF, Capacitor_SMD:C_1206_3216Metric_Pad1.33x1.80mm_HandSolder, F.Cu at (148.8, 156.9)
- added C203: 0.1uF, Capacitor_SMD:C_1206_3216Metric_Pad1.33x1.80mm_HandSolder, F.Cu at (164.9, 157.9)
- added C3: 4.7uF, Capacitor_SMD:C_1206_3216Metric_Pad1.33x1.80mm_HandSolder, F.Cu at (144.4, 207.8)
- added C300: 22uF, Capacitor_SMD:C_1206_3216Metric_Pad1.33x1.80mm_HandSolder, F.Cu at (150.9, 147.8)
- added C301: 2.2uF, Capacitor_SMD:C_1206_3216Metric_Pad1.33x1.80mm_HandSolder, F.Cu at (160.9, 135.7)
- added C302: 33pF, Capacitor_SMD:C_1206_3216Metric_Pad1.33x1.80mm_HandSolder, F.Cu at (150.9, 140.5)
- added C303: 33pF, Capacitor_SMD:C_1206_3216Metric_Pad1.33x1.80mm_HandSolder, F.Cu at (150.9, 136.6)
- added C4: 1uF, Capacitor_SMD:C_1206_3216Metric_Pad1.33x1.80mm_HandSolder, F.Cu at (144.6, 202.4)
- added C400: 22uF, Capacitor_SMD:C_1206_3216Metric_Pad1.33x1.80mm_HandSolder, F.Cu at (158.6, 203.1)
- added C401: 2.2uF, Capacitor_SMD:C_1206_3216Metric_Pad1.33x1.80mm_HandSolder, F.Cu at (168.8, 191.8)
- added C402: 33pF, Capacitor_SMD:C_1206_3216Metric_Pad1.33x1.80mm_HandSolder, F.Cu at (151.9, 198.7)
- added C403: 33pF, Capacitor_SMD:C_1206_3216Metric_Pad1.33x1.80mm_HandSolder, F.Cu at (151.9, 194.8)
- added C500: 0.1uF, Capacitor_SMD:C_1206_3216Metric_Pad1.33x1.80mm_HandSolder, F.Cu at (168.7, 181.0)
- added C501: 0.1uF, Capacitor_SMD:C_1206_3216Metric_Pad1.33x1.80mm_HandSolder, F.Cu at (168.7, 177.6)
- added C800: 100pF, Capacitor_SMD:C_1206_3216Metric_Pad1.33x1.80mm_HandSolder, F.Cu at (135.3, 204.1)
- added C900: 100pF, Capacitor_SMD:C_1206_3216Metric_Pad1.33x1.80mm_HandSolder, F.Cu at (117.1, 207.7)
- added D1: 2.0V, Diode_SMD:D_SOD-123, F.Cu at (150.1, 151.8)
- added D2: LED, LED_SMD:LED_1206_3216Metric_Pad1.42x1.75mm_HandSolder, F.Cu at (115.6, 189.8)
- added D300: BYG20J-E3/TR, Diode_SMD:D_SMA, F.Cu at (165.7, 153.3)
- added D301: MBRM130LT1G, SnapEDA Library:MBRM130LT1G, F.Cu at (173.9, 135.4)
- added D302: MBRM130LT1G, SnapEDA Library:MBRM130LT1G, F.Cu at (170.0, 147.2)
- added D400: BYG20J-E3/TR, Diode_SMD:D_SMA, F.Cu at (168.3, 187.4)
- added D401: MBRM130LT1G, SnapEDA Library:MBRM130LT1G, F.Cu at (170.9, 208.8)
- added D402: MBRM130LT1G, SnapEDA Library:MBRM130LT1G, F.Cu at (174.2, 201.1)
- added D500: CMOD4448 TR PBFREE, Diode_SMD:D_SOD-523, F.Cu at (159.3, 172.8)
- added FB1: MountingHole_Pad, TestPoint:TestPoint_THTPad_D2.5mm_Drill1.2mm, F.Cu at (140.9, 173.5)
- added GND1: MountingHole_Pad, MountingHole:MountingHole_8.4mm_M8_Pad_TopBottom, F.Cu at (82.2, 197.2)
- added GND2: MountingHole_Pad, TestPoint:TestPoint_THTPad_D2.5mm_Drill1.2mm, F.Cu at (138.2, 144.5)
- added IC2: MAX1681ESA+, SnapEDA Library:SOIC127P600X175-8N, F.Cu at (126.0, 202.5)
- added IC4: AD8092ARZ, SnapEDA Library:SOIC127P600X175-8N, F.Cu at (126.0, 195.7)
- added L4: 22uH, SnapEDA Library:IND_MSS1210_COC, F.Cu at (130.3, 176.7)
- added ON/OFF1: MountingHole_Pad, TestPoint:TestPoint_THTPad_D2.5mm_Drill1.2mm, F.Cu at (138.5, 154.8)
- added Q33: DMT10H009LK3-13, SnapEDA Library:TO-252-3_TabPin2 modded, F.Cu at (131.9, 163.1)
- added Q34: DMT10H009LK3-13, SnapEDA Library:TO-252-3_TabPin2 modded, F.Cu at (115.2, 169.3)
- added R100: 62.0k, Resistor_SMD:R_1206_3216Metric_Pad1.30x1.75mm_HandSolder, F.Cu at (133.2, 148.0)
- added R101: 4.99k, Resistor_SMD:R_1206_3216Metric_Pad1.30x1.75mm_HandSolder, F.Cu at (116.4, 145.3)
- added R102: 39.2k, Resistor_SMD:R_1206_3216Metric_Pad1.30x1.75mm_HandSolder, F.Cu at (127.6, 145.3)
- added R103: 20k, Resistor_SMD:R_1206_3216Metric_Pad1.30x1.75mm_HandSolder, F.Cu at (120.1, 145.3)
- added R104: 20k, Resistor_SMD:R_1206_3216Metric_Pad1.30x1.75mm_HandSolder, F.Cu at (118.1, 151.4)
- added R105: 866, Resistor_SMD:R_1206_3216Metric_Pad1.30x1.75mm_HandSolder, F.Cu at (112.8, 157.5)
- added R106: 2.87k, Resistor_SMD:R_1206_3216Metric_Pad1.30x1.75mm_HandSolder, F.Cu at (119.5, 137.2)
- added R107: 1.27k, Resistor_SMD:R_1206_3216Metric_Pad1.30x1.75mm_HandSolder, F.Cu at (115.9, 137.2)
- added R108: 18k, Resistor_SMD:R_1206_3216Metric_Pad1.30x1.75mm_HandSolder, F.Cu at (120.0, 184.2)
- added R109: 24.9, Resistor_SMD:R_1206_3216Metric_Pad1.30x1.75mm_HandSolder, F.Cu at (116.5, 184.2)
- added R110: 1k, Resistor_SMD:R_1206_3216Metric_Pad1.30x1.75mm_HandSolder, F.Cu at (122.4, 189.8)
- added R200: 30.1k, Resistor_SMD:R_1206_3216Metric_Pad1.30x1.75mm_HandSolder, F.Cu at (158.4, 165.8)
- added R201: 36.5k, Resistor_SMD:R_1206_3216Metric_Pad1.30x1.75mm_HandSolder, F.Cu at (171.5, 159.9)
- added R202: 1.37k, Resistor_SMD:R_1206_3216Metric_Pad1.30x1.75mm_HandSolder, F.Cu at (167.9, 163.2)
- added R203: 2.0k, Resistor_SMD:R_1206_3216Metric_Pad1.30x1.75mm_HandSolder, F.Cu at (157.4, 153.7)
- added R204: 2.0k, Resistor_SMD:R_1206_3216Metric_Pad1.30x1.75mm_HandSolder, F.Cu at (152.3, 156.9)
- added R3: 10k, Resistor_SMD:R_1206_3216Metric_Pad1.30x1.75mm_HandSolder, F.Cu at (141.3, 178.7)
- added R300: 49.9, Resistor_SMD:R_1206_3216Metric_Pad1.30x1.75mm_HandSolder, F.Cu at (156.8, 148.5)
- added R301: 3.3, Resistor_SMD:R_1206_3216Metric_Pad1.30x1.75mm_HandSolder, F.Cu at (170.3, 138.2)
- added R302: 3.3, Resistor_SMD:R_1206_3216Metric_Pad1.30x1.75mm_HandSolder, F.Cu at (168.8, 141.9)
- added R304: 150, Resistor_SMD:R_1206_3216Metric_Pad1.30x1.75mm_HandSolder, F.Cu at (150.9, 144.2)
- added R305: 2.2, Resistor_SMD:R_1206_3216Metric_Pad1.30x1.75mm_HandSolder, F.Cu at (167.9, 134.5)
- added R306: 2.2, Resistor_SMD:R_1206_3216Metric_Pad1.30x1.75mm_HandSolder, F.Cu at (164.1, 146.3)
- added R400: 49.9, Resistor_SMD:R_1206_3216Metric_Pad1.30x1.75mm_HandSolder, F.Cu at (158.6, 206.8)
- added R401: 150, Resistor_SMD:R_1206_3216Metric_Pad1.30x1.75mm_HandSolder, F.Cu at (151.9, 202.4)
- added R403: 3.3, Resistor_SMD:R_1206_3216Metric_Pad1.30x1.75mm_HandSolder, F.Cu at (168.2, 203.8)
- added R404: 3.3, Resistor_SMD:R_1206_3216Metric_Pad1.30x1.75mm_HandSolder, F.Cu at (169.8, 196.3)
- added R405: 2.2, Resistor_SMD:R_1206_3216Metric_Pad1.30x1.75mm_HandSolder, F.Cu at (165.0, 207.8)
- added R406: 2.2, Resistor_SMD:R_1206_3216Metric_Pad1.30x1.75mm_HandSolder, F.Cu at (168.2, 200.1)
- added R504: 150, Resistor_SMD:R_1206_3216Metric_Pad1.30x1.75mm_HandSolder, F.Cu at (160.5, 169.5)
- added R505: 150, Resistor_SMD:R_1206_3216Metric_Pad1.30x1.75mm_HandSolder, F.Cu at (159.1, 185.8)
- added R506: 150, Resistor_SMD:R_1206_3216Metric_Pad1.30x1.75mm_HandSolder, F.Cu at (152.3, 169.8)
- added R507: 150, Resistor_SMD:R_1206_3216Metric_Pad1.30x1.75mm_HandSolder, F.Cu at (159.1, 189.3)
- added R508: 150, Resistor_SMD:R_1206_3216Metric_Pad1.30x1.75mm_HandSolder, F.Cu at (150.8, 178.1)
- added R509: 150, Resistor_SMD:R_1206_3216Metric_Pad1.30x1.75mm_HandSolder, F.Cu at (150.8, 174.6)
- added R510: 1k, Resistor_SMD:R_1206_3216Metric_Pad1.30x1.75mm_HandSolder, F.Cu at (152.4, 183.6)
- added R511: 1k, Resistor_SMD:R_1206_3216Metric_Pad1.30x1.75mm_HandSolder, F.Cu at (145.4, 189.2)
- added R800: 1k, Resistor_SMD:R_1206_3216Metric_Pad1.30x1.75mm_HandSolder, F.Cu at (241.1, 242.6)
- added R801: 1k, Resistor_SMD:R_1206_3216Metric_Pad1.30x1.75mm_HandSolder, F.Cu at (239.5, 206.3)
- added R802: 0.0001, SnapEDA Library:PSR500HTQFB0L10, F.Cu at (151.0, 255.6)
- added R803: 300, Resistor_SMD:R_1206_3216Metric_Pad1.30x1.75mm_HandSolder, F.Cu at (137.7, 207.8)
- added R804: 10k, Resistor_SMD:R_1206_3216Metric_Pad1.30x1.75mm_HandSolder, F.Cu at (135.3, 200.4)
- added R805: 148k, Resistor_SMD:R_1206_3216Metric_Pad1.30x1.75mm_HandSolder, F.Cu at (132.9, 195.4)
- added R900: 1k, Resistor_SMD:R_1206_3216Metric_Pad1.30x1.75mm_HandSolder, F.Cu at (241.1, 96.8)
- added R901: 1k, Resistor_SMD:R_1206_3216Metric_Pad1.30x1.75mm_HandSolder, F.Cu at (239.5, 133.1)
- added R902: 0.0001, SnapEDA Library:PSR500HTQFB0L10, F.Cu at (151.0, 83.8)
- added R903: 300, Resistor_SMD:R_1206_3216Metric_Pad1.30x1.75mm_HandSolder, F.Cu at (117.1, 204.1)
- added R904: 10k, Resistor_SMD:R_1206_3216Metric_Pad1.30x1.75mm_HandSolder, F.Cu at (117.1, 200.4)
- added R905: 148k, Resistor_SMD:R_1206_3216Metric_Pad1.30x1.75mm_HandSolder, F.Cu at (118.5, 195.4)
- added U1: LM5032MTCX_NOPB, SnapEDA Library:SOP65P640X120-16N, F.Cu at (160.5, 177.8)
- added U2: LM8261M5, Package_TO_SOT_SMD:SOT-23-5, F.Cu at (157.9, 157.8)
- added U3: UCC27712DR, SnapEDA Library:SOIC127P599X175-8N, F.Cu at (159.8, 141.1)
- added U4: SN74LVC2G14IDCKRQ1, SnapEDA Library:SOT65P210X110-6N, F.Cu at (152.3, 189.1)
- added U5: UCC27712DR, SnapEDA Library:SOIC127P599X175-8N, F.Cu at (160.8, 196.1)
- added U6: LM5146QRGYRQ1, SnapEDA Library:QFN50P450X350X100-21N MODDED, F.Cu at (125.3, 152.4)
- added U7: SN74LVC2G08QDCURQ1, SnapEDA Library:U_VSSOP8_DCU_00_TEX, F.Cu at (145.9, 184.8)
- added U8: TPS76650DRM3, SnapEDA Library:D8, F.Cu at (143.3, 197.0)
- added V_IN1: MountingHole_Pad, MountingHole:MountingHole_8.4mm_M8_Pad_TopBottom, F.Cu at (82.2, 142.2)
- added V_OUT1: MountingHole_Pad, MountingHole:MountingHole_8.4mm_M8_Pad_TopBottom, F.Cu at (253.4, 169.7)
- added Vsense1: MountingHole_Pad, TestPoint:TestPoint_THTPad_D2.5mm_Drill1.2mm, F.Cu at (138.3, 139.5)
- L1, L2: footprint Library:IHDM1107BBEVR47M20 Inductor -> SnapEDA Library:EDITED-IND_IHDM1107BBEVR47M20_VIS
- Q1, Q10, Q11, Q12, Q13, Q14, Q15, Q16, Q2, Q3, Q4, Q5, Q6, Q7, Q8, Q9: footprint Package_TO_SOT_THT:TO-220-3_Vertical -> SnapEDA Library:TO-220-3_Horizontal_TabDown no hole
- R1: value R -> 47k
- R2: value R -> 1k
- R500: renamed from R6; value 50k -> 35.7k
- R501: renamed from R5; value 3.72k -> 1.1k
- moved Q13 195.4 mm to (183.4, 244.5)
- moved Q16 194.3 mm to (228.4, 244.5)
- moved Q14 193.7 mm to (198.4, 244.5)
- moved Q15 193.3 mm to (213.4, 244.5)
- moved C15 182.0 mm to (261.9, 196.0), turned to -90 degrees
- moved C8 175.8 mm to (257.4, 196.0), turned to -90 degrees
- moved C9 169.7 mm to (252.9, 196.0), turned to -90 degrees
- moved C10 163.6 mm to (248.4, 196.0), turned to -90 degrees
- moved Q12 160.1 mm to (228.4, 208.2)
- moved L2 159.6 mm to (147.0, 231.0), turned to 90 degrees
- moved Q11 156.0 mm to (213.4, 208.2)
- moved Q10 153.5 mm to (198.4, 208.2)
- moved Q9 152.7 mm to (183.4, 208.2)
- moved Q1 140.6 mm to (233.4, 131.2), turned to 180 degrees
- moved C14 127.4 mm to (261.9, 143.3), turned to 90 degrees
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- renumbered C4 to C15, R4 to R502, R3 to R503
Connections:
- Q1 pad 1: Net-(D2-A) -> Vout
- Q1 pad 2: Net-(Q1-G) -> /HO1
- Q1 pad 3: GND -> Net-(Q1-S)
- Q10 pad 1: Net-(D1-A) -> Vout
- Q10 pad 2: Net-(Q10-G) -> /HO2
- Q10 pad 3: GND -> Net-(Q10-S)
- Q11 pad 1: Net-(D1-A) -> Vout
- Q11 pad 2: Net-(Q10-G) -> /HO2
- Q11 pad 3: GND -> Net-(Q10-S)
- Q12 pad 1: Net-(D1-A) -> Vout
- Q12 pad 2: Net-(Q10-G) -> /HO2
- Q12 pad 3: GND -> Net-(Q10-S)
- Q13 pad 1: Net-(D1-A) -> Net-(Q10-S)
- Q13 pad 2: Net-(Q10-G) -> /LO2
- Q13 pad 3: GND -> Net-(Q13-S)
- Q14 pad 1: Net-(D1-A) -> Net-(Q10-S)
- Q14 pad 2: Net-(Q10-G) -> /LO2
- Q14 pad 3: GND -> Net-(Q13-S)
- Q15 pad 1: Net-(D1-A) -> Net-(Q10-S)
- Q15 pad 2: Net-(Q10-G) -> /LO2
- Q15 pad 3: GND -> Net-(Q13-S)
- Q16 pad 1: Net-(D1-A) -> Net-(Q10-S)
- Q16 pad 2: Net-(Q10-G) -> /LO2
- Q16 pad 3: GND -> Net-(Q13-S)
- Q2 pad 1: Net-(D2-A) -> Vout
- Q2 pad 2: Net-(Q1-G) -> /HO1
- Q2 pad 3: GND -> Net-(Q1-S)
- Q3 pad 1: Net-(D2-A) -> Vout
- Q3 pad 2: Net-(Q1-G) -> /HO1
- Q3 pad 3: GND -> Net-(Q1-S)
- Q4 pad 1: Net-(D2-A) -> Vout
- Q4 pad 2: Net-(Q1-G) -> /HO1
- Q4 pad 3: GND -> Net-(Q1-S)
- Q5 pad 1: Net-(D2-A) -> Net-(Q1-S)
- Q5 pad 2: Net-(Q1-G) -> /LO1
- Q5 pad 3: GND -> Net-(Q5-S)
- Q6 pad 1: Net-(D2-A) -> Net-(Q1-S)
- Q6 pad 2: Net-(Q1-G) -> /LO1
- Q6 pad 3: GND -> Net-(Q5-S)
- Q7 pad 1: Net-(D2-A) -> Net-(Q1-S)
- Q7 pad 2: Net-(Q1-G) -> /LO1
- Q7 pad 3: GND -> Net-(Q5-S)
- Q8 pad 1: Net-(D2-A) -> Net-(Q1-S)
- Q8 pad 2: Net-(Q1-G) -> /LO1
- Q8 pad 3: GND -> Net-(Q5-S)
- Q9 pad 1: Net-(D1-A) -> Vout
- Q9 pad 2: Net-(Q10-G) -> /HO2
- Q9 pad 3: GND -> Net-(Q10-S)
- R1 pad 1: Vout -> Net-(ON/OFF1-Pad1)
- R1 pad 2: Net-(U2-NEG) -> Net-(U1-UVLO)
- R2 pad 1: Net-(U2-NEG) -> Net-(R2-Pad1)
- R2 pad 2: GND -> Vin
Routing:
- net /LO2: track 0.00 -> 214.6 mm
- net /LO1: track 0.00 -> 207.5 mm
- net Net-(Q5-S): track 0.00 -> 166.1 mm, vias 0 -> 59
- net /12V: track 0.00 -> 144.2 mm, vias 0 -> 7
- net /HO2: track 0.00 -> 100.8 mm
- net /HO1: track 0.00 -> 94.5 mm
- net /CS1: track 0.00 -> 92.1 mm, vias 0 -> 2
- net /5V: track 0.00 -> 86.4 mm, vias 0 -> 3
- net Vout: track 0.00 -> 81.4 mm, vias 0 -> 40
- net Net-(Q13-S): track 0.00 -> 78.7 mm, vias 0 -> 57
- net Net-(U3-LL): track 0.00 -> 71.5 mm, vias 0 -> 2
- net /CS2: track 0.00 -> 65.7 mm, vias 0 -> 2
- net Net-(U6-FB): track 0.00 -> 58.2 mm, vias 0 -> 3
- net Net-(U1-UVLO): track 0.00 -> 54.6 mm, vias 0 -> 2
- net GND: track 0.00 -> 52.6 mm, vias 0 -> 175
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- added copper zone on F.Cu, net /12V
- added copper zone on B.Cu, net GND
- added copper zone on F.Cu, net GND
- added copper zone on F.Cu, net Net-(D1-K)
- added copper zone on F.Cu, net Net-(D302-K)
- added copper zone on B.Cu, net Net-(Q1-S)
- added copper zone on F.Cu, net Net-(Q1-S)
- added copper zone on B.Cu, net Net-(Q10-S)
- added copper zone on F.Cu, net Net-(Q10-S)
- added copper zone on B.Cu, net Net-(Q13-S)
- added copper zone on F.Cu, net Net-(Q13-S)
- added copper zone on F.Cu, net Net-(Q33-S)
- added copper zone on B.Cu, net Net-(Q5-S)
- added copper zone on F.Cu, net Net-(Q5-S)
- added copper zone on F.Cu, net Net-(U6-EN_UVLO)
- added copper zone on F.Cu, net Vin
- added copper zone on B.Cu, net Vout
- added copper zone on F.Cu, net Vout
Other:
- board outline added: 200 x 200 mm
