File: LM5032 Boost Converter Sch.kicad_sch (KiCad schematic)
At the start: 24 parts, among them Q1 NMOS, Q2 NMOS, U1 LM5032MTCX_NOPB, U2 LM8261M5

Commit message: update
Parts:
- removed R7, R8: 0.02, symbol Device:R
- added C10, C11, C12, C13, C14, C8, C9: 10uF, Capacitor_SMD:C_1210_3225Metric_Pad1.33x2.70mm_HandSolder, symbol Device:C
- added Q10, Q11, Q12, Q13, Q14, Q15, Q16, Q3, Q4, Q5, Q6, Q7, Q8, Q9: NMOS, Package_TO_SOT_THT:TO-220-3_Vertical, symbol Simulation_SPICE:NMOS
- C4: value C -> 10uF; footprint (none) -> Capacitor_SMD:C_1210_3225Metric_Pad1.33x2.70mm_HandSolder
- L1, L2: footprint (none) -> Library:IHDM1107BBEVR47M20 Inductor
- Q1, Q2: footprint (none) -> Package_TO_SOT_THT:TO-220-3_Vertical
- R1, R2, R3, R4, R5, R6: footprint (none) -> Resistor_SMD:R_1206_3216Metric_Pad1.30x1.75mm_HandSolder
Connections:
- net GND: now also Q1.3 (S), Q2.3 (S), C10.2, C11.2, C12.2, C13.2, C14.2, C8.2, C9.2, Q10.3 (S), Q11.3 (S), Q12.3 (S), Q13.3 (S), Q14.3 (S), Q15.3 (S), Q16.3 (S), Q3.3 (S), Q4.3 (S), Q5.3 (S), Q6.3 (S), Q7.3 (S), Q8.3 (S), Q9.3 (S)
- net Vout: now also C10.1, C11.1, C12.1, C13.1, C14.1, C8.1, C9.1
- net at U1.3 (CS1): no longer Q2.3 (S)
- net at D2.2 (A), L2.2, Q1.1 (D): now also Q2.1 (D), Q3.1 (D), Q4.1 (D), Q5.1 (D), Q6.1 (D), Q7.1 (D), Q8.1 (D)
- net at Q1.2 (G), U1.10 (OUT2): now also Q2.2 (G), Q3.2 (G), Q4.2 (G), Q5.2 (G), Q6.2 (G), Q7.2 (G), Q8.2 (G)
- net at U1.13 (CS2): no longer Q1.3 (S)
- net at U1.7 (OUT1): now also Q10.2 (G), Q11.2 (G), Q12.2 (G), Q13.2 (G), Q14.2 (G), Q15.2 (G), Q16.2 (G), Q9.2 (G); no longer Q2.2 (G)
- net at D1.2 (A), L1.2: now also Q10.1 (D), Q11.1 (D), Q12.1 (D), Q13.1 (D), Q14.1 (D), Q15.1 (D), Q16.1 (D), Q9.1 (D); no longer Q2.1 (D)
Other:
- moved on the sheet: C1, C2, C3, C4, C5, C6, C7, D1, D2, D3, L1, L2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

Commit message: 'update'
Parts:
- removed D1, D2: D, symbol Device:D
- added C15, C16: 1uF, symbol Device:C
- added C17: 10nF, symbol Device:C
- added C18: 7.5nF, symbol Device:C
- added C19: 10uF, symbol Device:C
- added C20: 470pF, symbol Device:C
- added C21, C22, C23, C24: 0.1uF, symbol Device:C
- added L3: 390uH, Library:IHDM1107BBEVR47M20 Inductor, symbol Device:L
- added Q17, Q18, Q19, Q20, Q21, Q22, Q23, Q24, Q25, Q26, Q27, Q28, Q29, Q30, Q31, Q32: NMOS, Package_TO_SOT_THT:TO-220-3_Vertical, symbol Simulation_SPICE:NMOS
- added R10: 10k, Resistor_SMD:R_1206_3216Metric_Pad1.30x1.75mm_HandSolder, symbol Device:R
- added R11: 909, Resistor_SMD:R_1206_3216Metric_Pad1.30x1.75mm_HandSolder, symbol Device:R
- added R12: 2.49, Resistor_SMD:R_1206_3216Metric_Pad1.30x1.75mm_HandSolder, symbol Device:R
- added R13: 30.1k, Resistor_SMD:R_1206_3216Metric_Pad1.30x1.75mm_HandSolder, symbol Device:R
- added R14: 4.75k, Resistor_SMD:R_1206_3216Metric_Pad1.30x1.75mm_HandSolder, symbol Device:R
- added R15, R16, R17, R18: 1, Resistor_SMD:R_1206_3216Metric_Pad1.30x1.75mm_HandSolder, symbol Device:R
- added R19, R20, R21, R22: 1k, Resistor_SMD:R_1206_3216Metric_Pad1.30x1.75mm_HandSolder, symbol Device:R
- added R23, R24, R25, R26: 49.9, Resistor_SMD:R_1206_3216Metric_Pad1.30x1.75mm_HandSolder, symbol Device:R
- added R7: 365k, Resistor_SMD:R_1206_3216Metric_Pad1.30x1.75mm_HandSolder, symbol Device:R
- added R8: 56.2k, Resistor_SMD:R_1206_3216Metric_Pad1.30x1.75mm_HandSolder, symbol Device:R
- added R9: 6.34k, Resistor_SMD:R_1206_3216Metric_Pad1.30x1.75mm_HandSolder, symbol Device:R
- added U3, U5: UCC27712DR, SnapEDA Library:SOIC127P599X175-8N, symbol UCC27712DR:UCC27712DR
- added U4: LM5018MR_NOPB, SnapEDA Library:VREG_LM5017MR_NOPB, symbol LM5018MR_NOPB:LM5018MR_NOPB
Connections:
- net Vsupply is gone; now on net 15V: U2.5 (V+)
- net GND: now also C15.2, C16.2, C22.1, C23.1, C24.1, Q25.3 (S), Q26.3 (S), Q27.3 (S), Q28.3 (S), Q29.3 (S), Q30.3 (S), Q31.3 (S), Q32.3 (S), R11.2, R12.2, R21.1, R22.1, R9.2, U4.1 (RTN); no longer Q1.3 (S), Q2.3 (S), Q3.3 (S), Q4.3 (S), Q5.3 (S), Q6.3 (S), Q7.3 (S), Q8.3 (S), U2.3 (POS)
- net Vin: now also C15.1, R7.1, R8.1, U4.2 (VIN); no longer U1.1 (VIN)
- net Vout: now also Q1.3 (S), Q10.1 (D), Q11.1 (D), Q12.1 (D), Q13.1 (D), Q14.1 (D), Q15.1 (D), Q16.1 (D), Q2.3 (S), Q3.3 (S), Q4.3 (S), Q5.3 (S), Q6.3 (S), Q7.3 (S), Q8.3 (S), Q9.1 (D), Q17.3 (S), Q18.3 (S), Q19.3 (S), Q20.3 (S), Q21.3 (S), Q22.3 (S), Q23.3 (S), Q24.3 (S), Q25.1 (D), Q26.1 (D), Q27.1 (D), Q28.1 (D), Q29.1 (D), Q30.1 (D), Q31.1 (D), Q32.1 (D), R19.1, R20.1, U3.6 (HS), U5.6 (HS)
- net LO1: now reaches Q10.2 (G), Q11.2 (G), Q12.2 (G), Q13.2 (G), Q14.2 (G), Q15.2 (G), Q16.2 (G), Q9.2 (G)
- net LO1: now also R16.1, R22.2; no longer U1.7 (OUT1)
- net at D3.1 (K), U2.1 (OUT): now also C20.1, R13.1
- net at R1.2, R2.1, U2.4 (NEG): now also C20.2, C21.2
- net at Q1.1 (D), Q2.1 (D), Q3.1 (D)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: now also L1.2; no longer L2.2
- net HO1: now reaches Q1.2 (G), Q2.2 (G), Q3.2 (G), Q4.2 (G), Q5.2 (G), Q6.2 (G), Q7.2 (G), Q8.2 (G)
- net HO1: now also R15.1, R19.2; no longer U1.10 (OUT2)
- net at U1.11 (RES): now also C23.2
- net at U1.12 (SS2): now also U1.4 (SS1), C24.2
- net 15V: now reaches U1.6 (VCC)
- net 15V: now also U1.1 (VIN), C18.1, C19.1, L3.2, R10.1
- new net: R26.2, U5.1 (LL)
- new net: R25.2, U5.2 (HL)
- new net: R18.2, U5.5 (LO)
- new net: R17.2, U5.7 (HO)
- new net: L2.2, Q17.1 (D), Q18.1 (D), Q19.1 (D), Q20.1 (D), Q21.1 (D), Q22.1 (D), Q23.1 (D), Q24.1 (D)
- new net: R7.2, U4.4 (RON)
- new net: C16.1, U4.6 (VCC)
- new net: R24.1, R25.1, U1.7 (OUT1)
- new net: R24.2, U3.1 (LL)
- new net: C22.2, U2.3 (POS)
- new net: R23.1, R26.1, U1.10 (OUT2)
- new net: R15.2, U3.7 (HO)
- new net: C18.2, R10.2, R11.1, U4.5 (FB)
- new net: C17.1, U4.7 (BST)
- new net: C17.2, L3.1, U4.8 (SW)
- new net: C21.1, R13.2
- new net: R23.2, U3.2 (HL)
- new net: R16.2, U3.5 (LO)
- new net: R8.2, R9.1, U4.3 (UVLO)
- new net: C19.2, R12.1
- new net HO2: Q17.2 (G), Q18.2 (G), Q19.2 (G), Q20.2 (G), Q21.2 (G), Q22.2 (G), Q23.2 (G), Q24.2 (G), R17.1, R20.2
- new net LO2: Q25.2 (G), Q26.2 (G), Q27.2 (G), Q28.2 (G), Q29.2 (G), Q30.2 (G), Q31.2 (G), Q32.2 (G), R18.1, R21.2
Other:
- moved on the sheet: C10, C11, C12, C13, C14, C4, C5, C6, C7, C8, C9, D3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

Commit message: update
Parts:
- removed C15: 1uF, symbol Device:C
- removed C5, C6, C7: C, symbol Device:C
- removed L3: 390uH, Library:IHDM1107BBEVR47M20 Inductor, symbol Device:L
- removed Q1, Q17, Q18, Q19, Q20, Q21, Q22, Q23, Q24, Q25, Q26, Q27, Q28, Q29, Q30, Q31, Q32: NMOS, Package_TO_SOT_THT:TO-220-3_Vertical, symbol Simulation_SPICE:NMOS
- removed R10: 10k, Resistor_SMD:R_1206_3216Metric_Pad1.30x1.75mm_HandSolder, symbol Device:R
- removed R11: 909, Resistor_SMD:R_1206_3216Metric_Pad1.30x1.75mm_HandSolder, symbol Device:R
- removed R12: 2.49, Resistor_SMD:R_1206_3216Metric_Pad1.30x1.75mm_HandSolder, symbol Device:R
- removed R14: 4.75k, Resistor_SMD:R_1206_3216Metric_Pad1.30x1.75mm_HandSolder, symbol Device:R
- removed R17, R18: 1, Resistor_SMD:R_1206_3216Metric_Pad1.30x1.75mm_HandSolder, symbol Device:R
- removed R24, R26: 49.9, Resistor_SMD:R_1206_3216Metric_Pad1.30x1.75mm_HandSolder, symbol Device:R
- removed R7: 365k, Resistor_SMD:R_1206_3216Metric_Pad1.30x1.75mm_HandSolder, symbol Device:R
- removed R8: 56.2k, Resistor_SMD:R_1206_3216Metric_Pad1.30x1.75mm_HandSolder, symbol Device:R
- removed R9: 6.34k, Resistor_SMD:R_1206_3216Metric_Pad1.30x1.75mm_HandSolder, symbol Device:R
- removed U4: LM5018MR_NOPB, SnapEDA Library:VREG_LM5017MR_NOPB, symbol LM5018MR_NOPB:LM5018MR_NOPB
- added C100: 10uF, Capacitor_SMD:C_1210_3225Metric_Pad1.33x2.70mm_HandSolder, symbol Device:C
- added C101, C104, C105: 100nF, Capacitor_SMD:C_1206_3216Metric_Pad1.33x1.80mm_HandSolder, symbol Device:C
- added C102: 56nF, Capacitor_SMD:C_1206_3216Metric_Pad1.33x1.80mm_HandSolder, symbol Device:C
- added C103, C301, C401: 2.2uF, Capacitor_SMD:C_1206_3216Metric_Pad1.33x1.80mm_HandSolder, symbol Device:C
- added C106: 8.2nF, Capacitor_SMD:C_1206_3216Metric_Pad1.33x1.80mm_HandSolder, symbol Device:C
- added C107: 470pF, Capacitor_SMD:C_1206_3216Metric_Pad1.33x1.80mm_HandSolder, symbol Device:C
- added C108: 820pF, Capacitor_SMD:C_1206_3216Metric_Pad1.33x1.80mm_HandSolder, symbol Device:C
- added C109, C300, C400: 22uF, Capacitor_SMD:C_1206_3216Metric_Pad1.33x1.80mm_HandSolder, symbol Device:C
- added C203: 0.1uF, Capacitor_SMD:C_1206_3216Metric_Pad1.33x1.80mm_HandSolder, symbol Device:C
- added C302, C303, C402, C403: 33pF, Capacitor_SMD:C_1206_3216Metric_Pad1.33x1.80mm_HandSolder, symbol Device:C
- added C4: 1uF, Capacitor_SMD:C_1206_3216Metric_Pad1.33x1.80mm_HandSolder, symbol Device:C
- added C800, C900: 100pF, Capacitor_SMD:C_1206_3216Metric_Pad1.33x1.80mm_HandSolder, symbol Device:C
- added D100: LED, LED_SMD:LED_1206_3216Metric_Pad1.42x1.75mm_HandSolder, symbol Device:LED
- added D200: 2.0V, Diode_SMD:D_SOD-123, symbol Device:D_Zener
- added D300, D400: BYG20J-E3/TR, Diode_SMD:D_SMA, symbol Device:D
- added D301, D302, D401, D402: MBRM130LT1G, SnapEDA Library:MBRM130LT1G, symbol MBRM130LT1G:MBRM130LT1G
- added FB1, GND2, ON/OFF1, Vsense1: MountingHole_Pad, TestPoint:TestPoint_THTPad_D2.5mm_Drill1.2mm, symbol Mechanical:MountingHole_Pad
- added GND1, V_IN1, V_OUT1: MountingHole_Pad, MountingHole:MountingHole_8.4mm_M8_Pad_TopBottom, symbol Mechanical:MountingHole_Pad
- added IC1: AD8092ARZ, SOIC127P600X175-8N, symbol AD8092ARZ:AD8092ARZ
- added IC2: MAX1681ESA+, SOIC127P600X175-8N, symbol MAX1681ESA+:MAX1681ESA+
- added L4: 22uH, SnapEDA Library:IND_MSS1210_COC, symbol Device:L
- added Q100, Q101: DMT10H009LK3-13, SnapEDA Library:TO-252-3_TabPin2 modded, symbol Simulation_SPICE:NMOS
- added Q5: NMOS, SnapEDA Library:TO-220-3_Horizontal_TabDown no hole, symbol Simulation_SPICE:NMOS
- added R100: 62.0k, Resistor_SMD:R_1206_3216Metric_Pad1.30x1.75mm_HandSolder, symbol Device:R
- added R101: 4.99k, Resistor_SMD:R_1206_3216Metric_Pad1.30x1.75mm_HandSolder, symbol Device:R
- added R102: 39.2k, Resistor_SMD:R_1206_3216Metric_Pad1.30x1.75mm_HandSolder, symbol Device:R
- added R103, R104: 20k, Resistor_SMD:R_1206_3216Metric_Pad1.30x1.75mm_HandSolder, symbol Device:R
- added R105: 866, Resistor_SMD:R_1206_3216Metric_Pad1.30x1.75mm_HandSolder, symbol Device:R
- added R106: 2.87k, Resistor_SMD:R_1206_3216Metric_Pad1.30x1.75mm_HandSolder, symbol Device:R
- added R107: 1.27k, Resistor_SMD:R_1206_3216Metric_Pad1.30x1.75mm_HandSolder, symbol Device:R
- added R108: 18k, Resistor_SMD:R_1206_3216Metric_Pad1.30x1.75mm_HandSolder, symbol Device:R
- added R109: 24.9, Resistor_SMD:R_1206_3216Metric_Pad1.30x1.75mm_HandSolder, symbol Device:R
- added R110, R610, R611: 1k, Resistor_SMD:R_1206_3216Metric_Pad1.30x1.75mm_HandSolder, symbol Device:R
- added R201: 36.5k, Resistor_SMD:R_1206_3216Metric_Pad1.30x1.75mm_HandSolder, symbol Device:R
- added R202: 1.37k, Resistor_SMD:R_1206_3216Metric_Pad1.30x1.75mm_HandSolder, symbol Device:R
- added R203, R204: 2.0k, Resistor_SMD:R_1206_3216Metric_Pad1.30x1.75mm_HandSolder, symbol Device:R
- added R3, R804, R904: 10k, Resistor_SMD:R_1206_3216Metric_Pad1.30x1.75mm_HandSolder, symbol Device:R
- added R300, R400: 49.9, Resistor_SMD:R_1206_3216Metric_Pad1.30x1.75mm_HandSolder, symbol Device:R
- added R305, R306, R405, R406: 2.2, Resistor_SMD:R_1206_3216Metric_Pad1.30x1.75mm_HandSolder, symbol Device:R
- added R403, R404: 3.3, Resistor_SMD:R_1206_3216Metric_Pad1.30x1.75mm_HandSolder, symbol Device:R
- added R504, R505, R506, R507, R508, R509: 150, Resistor_SMD:R_1206_3216Metric_Pad1.30x1.75mm_HandSolder, symbol Device:R
- added R802, R902: 0.0001, SnapEDA Library:PSR500HTQFB0L10, symbol Device:R
- added R803, R903: 300, Resistor_SMD:R_1206_3216Metric_Pad1.30x1.75mm_HandSolder, symbol Device:R
- added R805, R905: 148k, Resistor_SMD:R_1206_3216Metric_Pad1.30x1.75mm_HandSolder, symbol Device:R
- added U1: LM5146QRGYRQ1, SnapEDA Library:QFN50P450X350X100-21N MODDED, symbol 2024-03-17_20-51-26:LM5146QRGYRQ1
- added U6: SN74LVC2G14IDCKRQ1, SnapEDA Library:SOT65P210X110-6N, symbol SN74LVC2G14IDCKRQ1:SN74LVC2G14IDCKRQ1
- added U7: SN74LVC2G08QDCURQ1, U_VSSOP8_DCU_00_TEX, symbol SN74LVC2G08QDCURQ1:SN74LVC2G08QDCURQ1
- added U8: TPS76650DRM3, D8, symbol TPS76650DRM3:TPS76650DRM3
- C1, C2: value C -> 1uF; footprint (none) -> Capacitor_SMD:C_1206_3216Metric_Pad1.33x1.80mm_HandSolder
- C16: value 1uF -> 0.1uF; footprint (none) -> Capacitor_SMD:C_1210_3225Metric_Pad1.33x2.70mm_HandSolder
- C17: value 10nF -> 0.1uF; footprint (none) -> Capacitor_SMD:C_1210_3225Metric_Pad1.33x2.70mm_HandSolder
- C18: value 7.5nF -> 0.1uF; footprint (none) -> Capacitor_SMD:C_1210_3225Metric_Pad1.33x2.70mm_HandSolder
- C19: value 10uF -> 0.1uF; footprint (none) -> Capacitor_SMD:C_1210_3225Metric_Pad1.33x2.70mm_HandSolder
- C200: renamed from C20; footprint (none) -> Capacitor_SMD:C_1206_3216Metric_Pad1.33x1.80mm_HandSolder
- C201: renamed from C21; footprint (none) -> Capacitor_SMD:C_1206_3216Metric_Pad1.33x1.80mm_HandSolder
- C202: renamed from C22; footprint (none) -> Capacitor_SMD:C_1206_3216Metric_Pad1.33x1.80mm_HandSolder
- C3: value C -> 4.7uF; footprint (none) -> Capacitor_SMD:C_1206_3216Metric_Pad1.33x1.80mm_HandSolder
- C500: renamed from C23; footprint (none) -> Capacitor_SMD:C_1206_3216Metric_Pad1.33x1.80mm_HandSolder
- C501: renamed from C24; footprint (none) -> Capacitor_SMD:C_1206_3216Metric_Pad1.33x1.80mm_HandSolder
- D500: renamed from D3; value D -> CMOD4448 TR PBFREE; footprint (none) -> Diode_SMD:D_SOD-523
- L1, L2: footprint Library:IHDM1107BBEVR47M20 Inductor -> SnapEDA Library:EDITED-IND_IHDM1107BBEVR47M20_VIS
- Q1: renamed from Q5; footprint Package_TO_SOT_THT:TO-220-3_Vertical -> SnapEDA Library:TO-220-3_Horizontal_TabDown no hole
- Q10, Q11, Q12, Q13, Q14, Q15, Q16, Q2, Q3, Q4, Q6, Q7, Q8, Q9: footprint Package_TO_SOT_THT:TO-220-3_Vertical -> SnapEDA Library:TO-220-3_Horizontal_TabDown no hole
- R1: value R -> 5.36k (47k)
- R2: value R -> 1k
- R301: renamed from R15; value 1 -> 3.3
- R302: renamed from R16; value 1 -> 3.3
- R304: renamed from R23; value 49.9 -> 150
- R401: renamed from R25; value 49.9 -> 150
- R500: renamed from R6; value 50k -> 36.5k (35.7k)
- R501: renamed from R5; value 3.72k -> 1.1k
- R502: renamed from R4; value 28.7k -> 34.1k
- U2: footprint LM8261M5:SOT95P280X145-5N -> Package_TO_SOT_SMD:SOT-23-5
- U5: renamed from U1; footprint LM5032MTCX_NOPB:SOP65P640X120-16N -> SnapEDA Library:SOP65P640X120-16N
- renumbered C9 to C10, C10 to C11, C11 to C12, C12 to C13, C13 to C14, C14 to C15, C4 to C9, R13 to R200, R3 to R503, R21 to R800, R20 to R801, R22 to R900, R19 to R901, U5 to U4
Connections:
- net GND: now also C17.2, C18.2, C19.2, C2.1, U3.4 (COM), U4.4 (COM), C100.2, C101.2, C103.2, C105.2, C109.2, C203.1, C300.1, C302.1, C303.1, C4.1, C400.1, C402.1, C403.1, C800.1, C900.1, D100.1 (K), D200.2 (A), GND1.1, GND2.1, IC2.1 (FSEL), IC2.3 (GND), IC2.6 (LV), IC2.7 (SHDN), Q101.3 (S), R101.2, R107.2, R202.2, R506.2, R507.2, R509.1, R802.2, R804.2, R902.2, R904.2, U1.12 (PGND), U1.15 (EP), U1.16 (NC), U1.21 (EP), U1.6 (AGND), U1.9 (NC), U6.2 (GND), U7.4 (GND), U8.3 (GND), U8.4 (*EN); no longer C1.2, C2.2, Q10.3 (S), Q11.3 (S), Q12.3 (S), Q13.3 (S), Q14.3 (S), Q15.3 (S), Q16.3 (S), Q9.3 (S), R2.2, R800.1, R900.1
- net HO1: now also D301.2 (A); no longer Q6.2 (G), Q7.2 (G), Q8.2 (G)
- net HO2: now also Q10.2 (G), Q11.2 (G), Q12.2 (G), Q9.2 (G), D401.2 (A), R403.1
- net LO1: now also Q6.2 (G), Q7.2 (G), Q8.2 (G), D302.2 (A), Q5.2 (G); no longer Q10.2 (G), Q11.2 (G), Q12.2 (G), Q13.2 (G), Q14.2 (G), Q15.2 (G), Q16.2 (G), Q9.2 (G)
- net LO2: now also Q13.2 (G), Q14.2 (G), Q15.2 (G), Q16.2 (G), D402.2 (A), R404.1
- net Vin: now also R2.2, C100.1, C101.1, Q100.1 (D), R100.1, U1.20 (VIN), V_IN1.1; no longer C1.1, C2.1, C3.1
- net Vout: now also C16.1, C17.1, C18.1, C19.1, Q1.1 (D), Q2.1 (D), Q3.1 (D), Q4.1 (D), C301.2, C401.2, R201.1, V_OUT1.1; no longer Q1.3 (S), Q13.1 (D), Q14.1 (D), Q15.1 (D), Q16.1 (D), Q2.3 (S), Q3.3 (S), Q4.3 (S), Q6.3 (S), Q7.3 (S), Q8.3 (S), R1.1, R801.1, R901.1
- net at C200.2, C201.2, U2.4 (NEG): now also R201.2, R202.1; no longer R1.2, R2.1
- net at U4.1 (LL): now also C403.2, R504.2, R506.1, U6.3 (2A)
- net at R401.2, U4.2 (HL): now also C402.2
- net 12V: now reaches U4.3 (VDD)
- net 12V: now also U2.5 (V+), U3.3 (VDD), U5.1 (VIN), C109.1, C203.2, C300.2, C4.2, C400.2, L4.2, R108.1, R109.1, R110.1, R203.1, R300.2, R400.2, U8.5 (IN), U8.6 (IN)
- net at U4.5 (LO): now also R404.2, R406.2
- net at U4.7 (HO): now also R403.2, R405.2
- net at U4.8 (HB): now also C401.1, D400.1 (K)
- net at L2.2: now also Q10.3 (S), Q11.3 (S), Q12.3 (S), Q13.1 (D), Q14.1 (D), Q15.1 (D), Q16.1 (D), Q9.3 (S), R801.1
- net at R401.1: now also U7.3 (2Y); no longer U5.7 (OUT1)
- net at U3.1 (LL): now also C303.2, R505.2, R507.1, U6.1 (1A)
- net at C202.2, U2.3 (POS): now also R204.1
- net at R304.1: now also U7.7 (1Y); no longer U5.10 (OUT2)
- net at L1.2, Q6.1 (D), Q7.1 (D)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: now also Q1.3 (S), Q2.3 (S), Q3.3 (S), Q4.3 (S), R901.1, Q5.1 (D); no longer Q1.1 (D), Q2.1 (D), Q3.1 (D), Q4.1 (D)
- net at R500.2, R501.1, U5.5 (UVLO): now also R1.2
- net at R301.2, U3.7 (HO): now also R305.2
- net CS2: now reaches U5.13 (CS2)
- net CS2: now also IC1.7 (OUT), R805.1
- net CS1: now reaches U5.3 (CS1)
- net CS1: now also IC1.1 (OUT1), R905.1
- net at R304.2, U3.2 (HL): now also C302.2
- net at R302.2, U3.5 (LO): now also R306.2
- net at U3.8 (HB): now also C301.1, D300.1 (K)
- removed net 15V: C18.1, C19.1, U2.5 (V+), U5.1 (VIN), U5.6 (VCC)
- new net: R610.1, U6.4 (2Y)
- new net: R610.2, U7.6 (2B)
- new net: R508.2, U5.6 (VCC)
- new net: ON/OFF1.1, R1.1
- new net: IC1.2 (-IN1), R904.1, R905.2
- new net: C900.2, IC1.3 (+IN1), R903.1
- new net: R611.2, U7.2 (1B)
- new net: D300.2 (A), R300.1
- new net: C104.2, L4.1, Q100.3 (S), Q101.1 (D), R105.1, U1.19 (SW)
- new net: FB1.1, R3.1
- new net: C107.1, C108.2, R106.1, R107.1, R108.2, U1.5 (FB)
- new net: Q13.3 (S), Q14.3 (S), Q15.3 (S), Q16.3 (S), R800.1, R802.1, R803.2
- new net: C800.2, IC1.5 (+IN2), R803.1
- new net: IC1.6 (-IN2), R804.1, R805.2
- new net: D100.2 (A), R110.2
- new net: C108.1, R109.2
- new net: C106.1, R106.2
- new net: C106.2, C107.2, U1.4 (COMP)
- new net: Q5.3 (S), Q6.3 (S), Q7.3 (S), Q8.3 (S), R900.1, R902.1, R903.2
- new net: D200.1 (K), R203.2, R204.2
- new net: D302.1 (K), R306.1
- new net: D402.1 (K), R406.1
- new net: D401.1 (K), R405.1
- new net: R611.1, U6.6 (1Y)
- new net: R103.1, U1.8 (SYNCIN)
- new net: C102.2, C103.1, R102.2, R103.2, R104.2, U1.14 (VCC)
- new net: Q100.2 (G), U1.18 (HO)
- new net: R504.1, U5.10 (OUT2)
- new net: R505.1, U5.7 (OUT1)
- new net: C1.1, IC2.4 (CAP-)
- new net: C1.2, IC2.2 (CAP+)
- new net: R100.2, R101.1, U1.1 (EN_UVLO)
- new net: R104.1, U1.10 (PGOOD)
- new net: C105.1, R105.2, U1.11 (ILIM)
- new net: Q101.2 (G), U1.13 (LO)
- new net: C104.1, U1.17 (BST)
- new net: R102.1, U1.2 (RT)
- new net: C102.1, U1.3 (SS_TRK)
- new net: R2.1, Vsense1.1
- new net: D301.1 (K), R305.1
- new net: D400.2 (A), R400.1
- new net -5V: C2.2, IC1.4 (-VS), IC2.5 (OUT)
- new net 5V: C3.1, IC1.8 (+VS), IC2.8 (IN), U6.5 (VCC), U7.8 (VCC), U8.7 (OUT), U8.8 (OUT)
- new net U1-VCC: R3.2, R508.1, R509.2, U7.1 (1A), U7.5 (2A)
Other:
- note added: "This line (Comp 1 and Comp 2) needs to be at <1.5V or to sink >1.4mA (current going out of lm5032) when Vout exceeds max allowable voltage"
- note added: "This line (U2 Negative) needs to be at >2.0V when Vout exceeds max allowable voltage (55.29V)"
- note added: "UVLO (<1.20V) when Vin < 16.11V"
- note added: "UVLO (<1.25V) when Vin < 18V"
- note added: "if Vin < 18V, lm5032 off regardless of ON/OFF pin if Vin > 18V, lm5032 off unless ON/OFF pin ≥5V"
- note added: "lm5032 sinks about 17mA into each CS line (CS1 and CS2)"
- note added: "time delay of <160ns"
- note added: "time delay of <2.5ns with Vcc = 5V"
- note added: "time delay of <3.8ns with Vcc = 5V"
- moved on the sheet: C10, C11, C12, C13, C14, C15, C200, C201, C202, C500, C501, C8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
