File: LM5032 2 Board Design/LM5032 Control Board.kicad_pcb (KiCad board)
At the start: 4 copper layers, 114.2 x 118.6 mm, 98 parts, among them IC1 AD8092ARZ, IC2 MAX1681ESA+, Q100 DMT10H009LK3-13, Q101 DMT10H009LK3-13, U1 LM5146QRGYRQ1, U2 LM8261M5, U5 LM5032MTCX_NOPB, U6 SN74LVC2G14IDCKRQ1, U7 SN74LVC2G08QDCURQ1, U8 TPS76650DRM3

Commit message: update
Parts:
- added 12V1: MountingHole_Pad, TestPoint:TestPoint_THTPad_D2.5mm_Drill1.2mm, F.Cu at (406.8, 106.6)
- added 12V2: MountingHole_Pad, TestPoint:TestPoint_THTPad_D2.5mm_Drill1.2mm, F.Cu at (406.8, 238.8)
- added C100: 10uF, Capacitor_SMD:C_1210_3225Metric_Pad1.33x2.70mm_HandSolder, F.Cu at (439.3, 192.8)
- added C101: 100nF, Capacitor_SMD:C_1206_3216Metric_Pad1.33x1.80mm_HandSolder, F.Cu at (439.3, 188.7)
- added C102: 56nF, Capacitor_SMD:C_1206_3216Metric_Pad1.33x1.80mm_HandSolder, F.Cu at (455.7, 195.3)
- added C103: 2.2uF, Capacitor_SMD:C_1206_3216Metric_Pad1.33x1.80mm_HandSolder, F.Cu at (459.4, 195.3)
- added C104: 100nF, Capacitor_SMD:C_1206_3216Metric_Pad1.33x1.80mm_HandSolder, F.Cu at (450.8, 169.3)
- added C105: 100nF, Capacitor_SMD:C_1206_3216Metric_Pad1.33x1.80mm_HandSolder, F.Cu at (459.4, 180.4)
- added C106: 8.2nF, Capacitor_SMD:C_1206_3216Metric_Pad1.33x1.80mm_HandSolder, F.Cu at (444.9, 195.3)
- added C107: 470pF, Capacitor_SMD:C_1206_3216Metric_Pad1.33x1.80mm_HandSolder, F.Cu at (452.1, 187.8)
- added C108: 820pF, Capacitor_SMD:C_1206_3216Metric_Pad1.33x1.80mm_HandSolder, F.Cu at (454.2, 155.0)
- added C109: 22uF, Capacitor_SMD:C_1206_3216Metric_Pad1.33x1.80mm_HandSolder, F.Cu at (459.6, 148.9)
- added C5: 1uF, Capacitor_SMD:C_1206_3216Metric_Pad1.33x1.80mm_HandSolder, F.Cu at (116.6, 254.0)
- added C6: 10uF, Capacitor_SMD:C_1206_3216Metric_Pad1.33x1.80mm_HandSolder, F.Cu at (116.6, 257.4)
- added C7: 0.1uF, Capacitor_SMD:C_1206_3216Metric_Pad1.33x1.80mm_HandSolder, F.Cu at (110.7, 244.2)
- added C8: 0.1uF, Capacitor_SMD:C_1206_3216Metric_Pad1.33x1.80mm_HandSolder, F.Cu at (110.7, 247.6)
- added C9: 0.1uF, Capacitor_SMD:C_1206_3216Metric_Pad1.33x1.80mm_HandSolder, F.Cu at (110.7, 250.9)
- added D100: LED, LED_SMD:LED_1206_3216Metric_Pad1.42x1.75mm_HandSolder, F.Cu at (461.8, 155.0)
- added GND2: MountingHole_Pad, TestPoint:TestPoint_THTPad_D2.5mm_Drill1.2mm, F.Cu at (411.8, 238.8)
- added GND3: MountingHole_Pad, TestPoint:TestPoint_THTPad_D2.5mm_Drill1.2mm, F.Cu at (411.8, 106.6)
- added GND4: MountingHole_Pad, TestPoint:TestPoint_THTPad_D2.5mm_Drill1.2mm, F.Cu at (401.8, 101.6)
- added GND5: MountingHole_Pad, TestPoint:TestPoint_THTPad_D2.5mm_Drill1.2mm, F.Cu at (396.8, 101.6)
- added GND6: MountingHole_Pad, TestPoint:TestPoint_THTPad_D2.5mm_Drill1.2mm, F.Cu at (396.8, 243.8)
- added HL1: MountingHole_Pad, TestPoint:TestPoint_THTPad_D2.5mm_Drill1.2mm, F.Cu at (411.8, 111.6)
- added HL2: MountingHole_Pad, TestPoint:TestPoint_THTPad_D2.5mm_Drill1.2mm, F.Cu at (411.8, 243.8)
- added L4: 22uH, SnapEDA Library:IND_MSS1210_COC, F.Cu at (442.2, 156.4)
- added LL1: MountingHole_Pad, TestPoint:TestPoint_THTPad_D2.5mm_Drill1.2mm, F.Cu at (411.8, 101.6)
- added LL2: MountingHole_Pad, TestPoint:TestPoint_THTPad_D2.5mm_Drill1.2mm, F.Cu at (411.8, 233.8)
- added Q100: DMT10H009LK3-13, SnapEDA Library:TO-252-3_TabPin2 modded, F.Cu at (440.6, 170.0)
- added Q101: DMT10H009LK3-13, SnapEDA Library:TO-252-3_TabPin2 modded, F.Cu at (457.3, 163.8)
- added R100: 62.0k, Resistor_SMD:R_1206_3216Metric_Pad1.30x1.75mm_HandSolder, F.Cu at (439.3, 185.1)
- added R101: 4.99k, Resistor_SMD:R_1206_3216Metric_Pad1.30x1.75mm_HandSolder, F.Cu at (444.9, 187.8)
- added R102: 39.2k, Resistor_SMD:R_1206_3216Metric_Pad1.30x1.75mm_HandSolder, F.Cu at (448.5, 187.8)
- added R103: 20k, Resistor_SMD:R_1206_3216Metric_Pad1.30x1.75mm_HandSolder, F.Cu at (455.7, 187.8)
- added R104: 20k, Resistor_SMD:R_1206_3216Metric_Pad1.30x1.75mm_HandSolder, F.Cu at (459.4, 187.8)
- added R105: 866, Resistor_SMD:R_1206_3216Metric_Pad1.30x1.75mm_HandSolder, F.Cu at (458.1, 174.3)
- added R106: 2.87k, Resistor_SMD:R_1206_3216Metric_Pad1.30x1.75mm_HandSolder, F.Cu at (448.5, 195.3)
- added R107: 1.27k, Resistor_SMD:R_1206_3216Metric_Pad1.30x1.75mm_HandSolder, F.Cu at (452.1, 195.3)
- added R108: 18k, Resistor_SMD:R_1206_3216Metric_Pad1.30x1.75mm_HandSolder, F.Cu at (452.4, 148.9)
- added R109: 24.9, Resistor_SMD:R_1206_3216Metric_Pad1.30x1.75mm_HandSolder, F.Cu at (456.0, 148.9)
- added R110: 1k, Resistor_SMD:R_1206_3216Metric_Pad1.30x1.75mm_HandSolder, F.Cu at (463.1, 148.9)
- added REF**: MountingHole_3.2mm_M3, MountingHole:MountingHole_3.2mm_M3, F.Cu at (464.0, 125.4)
- added REF**: MountingHole_3.2mm_M3, MountingHole:MountingHole_3.2mm_M3, F.Cu at (412.0, 172.7)
- added REF**: MountingHole_3.2mm_M3, MountingHole:MountingHole_3.2mm_M3, F.Cu at (360.0, 125.4)
- added REF**: MountingHole_3.2mm_M3, MountingHole:MountingHole_3.2mm_M3, F.Cu at (360.0, 220.0)
- added REF**: MountingHole_3.2mm_M3, MountingHole:MountingHole_3.2mm_M3, F.Cu at (464.0, 220.0)
- added Rsense1: MountingHole_Pad, TestPoint:TestPoint_THTPad_D2.5mm_Drill1.2mm, F.Cu at (396.8, 111.6)
- added Rsense2: MountingHole_Pad, TestPoint:TestPoint_THTPad_D2.5mm_Drill1.2mm, F.Cu at (396.8, 106.6)
- added Rsense3: MountingHole_Pad, TestPoint:TestPoint_THTPad_D2.5mm_Drill1.2mm, F.Cu at (396.8, 233.8)
- added Rsense4: MountingHole_Pad, TestPoint:TestPoint_THTPad_D2.5mm_Drill1.2mm, F.Cu at (396.8, 238.8)
- added TEMP1: MountingHole_Pad, TestPoint:TestPoint_THTPad_D2.5mm_Drill1.2mm, F.Cu at (406.8, 111.6)
- added TEMP2: MountingHole_Pad, TestPoint:TestPoint_THTPad_D2.5mm_Drill1.2mm, F.Cu at (401.8, 106.6)
- added TEMP3: MountingHole_Pad, TestPoint:TestPoint_THTPad_D2.5mm_Drill1.2mm, F.Cu at (406.8, 101.6)
- added TEMP4: MountingHole_Pad, TestPoint:TestPoint_THTPad_D2.5mm_Drill1.2mm, F.Cu at (406.8, 233.8)
- added TEMP5: MountingHole_Pad, TestPoint:TestPoint_THTPad_D2.5mm_Drill1.2mm, F.Cu at (401.8, 238.8)
- added TEMP6: MountingHole_Pad, TestPoint:TestPoint_THTPad_D2.5mm_Drill1.2mm, F.Cu at (406.8, 243.8)
- added U1: LM5146QRGYRQ1, SnapEDA Library:QFN50P450X350X100-21N MODDED, F.Cu at (451.8, 180.7)
- added U3: STM32F042K6T6TR, SnapEDA Library:QFP80P900X900X160-32N, F.Cu at (120.2, 246.6)
- added U4: MCP1700T-3302E_MB, SnapEDA Library:MCP1700T-3302E_MB updated, F.Cu at (123.8, 257.7)
- added V_IN2: MountingHole_Pad, TestPoint:TestPoint_THTPad_D2.5mm_Drill1.2mm, F.Cu at (401.8, 111.6)
- added Vcap1: MountingHole_Pad, TestPoint:TestPoint_THTPad_D2.5mm_Drill1.2mm, F.Cu at (401.8, 233.8)
- added Vout1: MountingHole_Pad, TestPoint:TestPoint_THTPad_D2.5mm_Drill1.2mm, F.Cu at (401.8, 243.8)
- U8: value TPS76650DRM3 -> LM2937ES-5.0; footprint SnapEDA Library:D8 -> SnapEDA Library:TO254P1524X483-4N modded
- moved C3 89.2 mm to (78.8, 166.1)
- moved C4 88.2 mm to (78.9, 170.5)
- moved U8 85.1 mm to (78.3, 154.1)
Connections:
- U8 pad 1: unconnected-(U8-NC/FB-Pad1) -> /12V
- U8 pad 2: unconnected-(U8-PG-Pad2) -> GND
- U8 pad 3: GND -> /5V
Routing:
- net Net-(U1-FB): track 65.2 -> 130.4 mm, vias 4 -> 8
- net Net-(U1-VCC): track 38.3 -> 76.6 mm, vias 3 -> 6
- net Net-(Q100-S): track 32.3 -> 64.6 mm, vias 6 -> 12
- net /5V: track 39.4 -> 17.5 mm, vias 0 -> 1
- net Net-(U1-SS_TRK): track 18.2 -> 36.5 mm, vias 2 -> 4
- net Net-(U1-COMP): track 16.4 -> 32.7 mm, vias 2 -> 4
- net Net-(Q101-G): track 11.1 -> 22.1 mm
- net Net-(Q100-G): track 10.5 -> 21.0 mm
- net GND: track 29.6 -> 38.6 mm, vias 15 -> 22
- net Vin: track 8.67 -> 17.3 mm, vias 5 -> 10
- net Net-(U1-BST): track 8.35 -> 16.7 mm
- net Net-(U1-PGOOD): track 7.44 -> 14.9 mm
- net /12V: track 7.84 -> 0.60 mm, vias 5 -> 7
- net Net-(U1-ILIM): track 5.91 -> 11.8 mm
- net Net-(U1-SYNCIN): track 5.12 -> 10.2 mm
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- added copper zone on B.Cu, net (none)
- added copper zone on F.Cu, net (none)
- added copper zone on In1.Cu, net (none)
- added copper zone on In2.Cu, net (none)
Other:
- board size 114.2 x 118.6 mm -> 368.6 x 151.6 mm
