File: LM5032 2 Board Design/LM5032 Control Board.kicad_sch (KiCad schematic)
At the start: 93 parts, among them IC1 AD8092ARZ, IC2 MAX1681ESA+, Q100 DMT10H009LK3-13, Q101 DMT10H009LK3-13, U1 LM5146QRGYRQ1, U2 LM8261M5, U5 LM5032MTCX_NOPB, U6 SN74LVC2G14IDCKRQ1, U7 SN74LVC2G08QDCURQ1, U8 TPS76650DRM3

Commit message: update
Parts:
- removed FB1: MountingHole_Pad, TestPoint:TestPoint_THTPad_D2.5mm_Drill1.2mm, symbol Mechanical:MountingHole_Pad
- removed R3: 1k, Resistor_SMD:R_1206_3216Metric_Pad1.30x1.75mm_HandSolder, symbol Device:R
- removed U8: TPS76650DRM3, D8, symbol TPS76650DRM3:TPS76650DRM3
- added C10, C7, C8, C9: 0.1uF, Capacitor_SMD:C_1206_3216Metric_Pad1.33x1.80mm_HandSolder, symbol Device:C
- added C5: 1uF, Capacitor_SMD:C_1206_3216Metric_Pad1.33x1.80mm_HandSolder, symbol Device:C
- added C6: 10uF, Capacitor_SMD:C_1206_3216Metric_Pad1.33x1.80mm_HandSolder, symbol Device:C
- added IC3: SN65HVD234DR, SnapEDA Library:SOIC127P600X175-8N, symbol SN65HVD234DR:SN65HVD234DR
- added R10, R11, R12, R13, R14, R6, R7, R9: 10k, Resistor_SMD:R_1206_3216Metric_Pad1.30x1.75mm_HandSolder, symbol Device:R
- added R15: 18k, Resistor_SMD:R_1206_3216Metric_Pad1.30x1.75mm_HandSolder, symbol Device:R
- added R16, R17, R19: 1k, Resistor_SMD:R_1206_3216Metric_Pad1.30x1.75mm_HandSolder, symbol Device:R
- added R18: 2k, Resistor_SMD:R_1206_3216Metric_Pad1.30x1.75mm_HandSolder, symbol Device:R
- added R8: 120, Resistor_SMD:R_1206_3216Metric_Pad1.30x1.75mm_HandSolder, symbol Device:R
- added U3: STM32F042K6T6TR, SnapEDA Library:QFP80P900X900X160-32N, symbol STM32F042K6T6TR:STM32F042K6T6TR
- added U4: MCP1700T-3302E_MB, SnapEDA Library:MCP1700T-3302E_MB updated, symbol MCP1700T-3302E_MB:MCP1700T-3302E_MB
- added U8: LM2937ES-5.0, SnapEDA Library:TO254P1524X483-4N modded, symbol LM2937ES-5.0:LM2937ES-5.0
- added Y1: 830055663, 830055663, symbol 830055663:830055663
- R2: value 1k -> 18k
Connections:
- net 12V: now also U8.1 (VIN)
- net 5V: now also C5.2, U4.2 (VIN), U8.3 (VOUT)
- net GND: now also C10.1, C5.1, C6.1, C7.1, C8.1, C9.1, IC3.2 (GND), R16.2, R17.2, R19.2, R6.1, R7.1, U3.16 (VSS), U3.32 (VSS), U4.1 (GND), U8.2 (GND), Y1.2 (GND_&_LID_1), Y1.4 (GND_&_LID_2)
- net Vin: now also Vcap1.1; no longer R2.2
- net TEMP1: now reaches TEMP1.1
- net TEMP1: now also R9.1, U3.6 (PA0)
- net TEMP3: now reaches TEMP3.1
- net TEMP3: now also R11.1, U3.8 (PA2)
- net Vout1: now reaches R2.1
- net Vout1: no longer Vcap1.1
- net TEMP2: now reaches TEMP2.1
- net TEMP2: now also R10.1, U3.7 (PA1)
- net TEMP5: now reaches TEMP5.1
- net TEMP5: now also R13.1, U3.10 (PA4)
- net TEMP4: now reaches TEMP4.1
- net TEMP4: now also R12.1, U3.9 (PA3)
- net TEMP6: now reaches TEMP6.1
- net TEMP6: now also R14.1, U3.11 (PA5)
- net U5-VCC renamed FB1
- net FB1: now also R18.1
- new net: R15.2, R16.1, U3.12 (PA6)
- new net: IC3.5 (EN), R7.2
- new net: U3.3 (PF1-OSC_OUT), Y1.1 (CRYSTAL_1)
- new net: U3.2 (PF0-OSC_IN), Y1.3 (CRYSTAL_2)
- new net: R18.2, R19.1, U3.15 (PB1)
- new net: R17.1, R2.2, U3.14 (PB0)
- new net: IC3.8 (RS), R6.2
- new net 3.3V: C10.2, C6.2, C7.2, C8.2, C9.2, IC3.3 (VCC), R10.2, R11.2, R12.2, R13.2, R14.2, R9.2, U3.1 (VDD), U3.17 (VDDIO2), U3.5 (VDDA), U4.3 (VOUT)
- new net CAN RX: IC3.4 (R), U3.21 (PA11)
- new net CAN TX: IC3.1 (D), U3.22 (PA12)
- new net CANH: IC3.7 (CANH), R8.2
- new net CANL: IC3.6 (CANL), R8.1
- new net USART1 RX: U3.20 (PA10)
- new net USART1 TX: U3.19 (PA9)
- new net Vcap1: R15.1
Other:
- note added: "AD8092 short circuit current of 130mA"
- note added: "Input current of 6mA"
- note added: "LM8261 short circuit current of 53mA"
- note added: "Max Vss input current of 120mA"
- note added: "Max capable output current of 250mA"
- note added: "Max capable output current of 500mA"
- note added: "Max current draw of 120mA"
- note added: "Max current draw of 130mA + 0.01mA + 0.067mA + 53mA + 120mA = 303mA"
- note added: "max current of about 2*(5V / 1000) = 0.01mA"
- note added: "max current of about 2*(5V / 150) = 0.067mA"
- note added: "when FB1 = 7.7V, PA7 = 2.57V"
- note added: "when Vcap1 = 48V, PA6 = 2.53V"
- note added: "when Vout1 = 52V, PA7 = 2.74V"
- moved on the sheet: 12V1, C4, GND2, GND3, HL1, HL2, LL1, LL2, Rsense1, Rsense2, TEMP1, TEMP2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
