File: LM5032 2 Board Design/LM5032 Switching Board Copper Inlay.kicad_pcb (KiCad board)
At the start: 4 copper layers, 170 x 158.2 mm, 94 parts, among them Q1 NMOS, Q10 NMOS, Q11 NMOS, Q12 NMOS, Q13 NMOS, Q14 NMOS, Q15 NMOS, Q16 NMOS, Q2 NMOS, Q3 NMOS, Q4 NMOS, Q5 NMOS, Q6 NMOS, Q7 NMOS, Q8 NMOS, Q9 NMOS, U3 UCC27712DR, U4 UCC27712DR

Commit message: update
Parts:
- added REF**: MountingHole_5.3mm_M5, MountingHole:MountingHole_5.3mm_M5, F.Cu at (203.6, 111.3)
- added REF**: MountingHole_5.3mm_M5, MountingHole:MountingHole_5.3mm_M5, F.Cu at (203.6, 210.7)
- added RT2: 36.5k, Resistor_SMD:R_0603_1608Metric_Pad0.98x0.95mm_HandSolder, F.Cu at (174.7, 120.3)
- added RT2: 36.5k, Resistor_SMD:R_0603_1608Metric_Pad0.98x0.95mm_HandSolder, F.Cu at (159.4, 126.3)
- added RT3: 36.5k, Resistor_SMD:R_0603_1608Metric_Pad0.98x0.95mm_HandSolder, F.Cu at (177.5, 155.9)
- added RT3: 36.5k, Resistor_SMD:R_0603_1608Metric_Pad0.98x0.95mm_HandSolder, F.Cu at (185.9, 156.5)
- added RT5: 36.5k, Resistor_SMD:R_0603_1608Metric_Pad0.98x0.95mm_HandSolder, F.Cu at (174.7, 201.8)
- added RT5: 36.5k, Resistor_SMD:R_0603_1608Metric_Pad0.98x0.95mm_HandSolder, F.Cu at (159.4, 195.8)
- added RT6: 36.5k, Resistor_SMD:R_0603_1608Metric_Pad0.98x0.95mm_HandSolder, F.Cu at (185.9, 165.5)
- added RT6: 36.5k, Resistor_SMD:R_0603_1608Metric_Pad0.98x0.95mm_HandSolder, F.Cu at (177.5, 166.1)
- REF**: value MountingHole_4.3mm_M4 -> MountingHole_5.3mm_M5; footprint MountingHole:MountingHole_4.3mm_M4 -> MountingHole:MountingHole_5.3mm_M5
- REF** (x4): value MountingHole_4.3mm_M4 -> MountingHole_3.2mm_M3; footprint MountingHole:MountingHole_4.3mm_M4 -> MountingHole:MountingHole_3.2mm_M3
- moved RT5 54.6 mm to (159.4, 192.4)
- moved RT2 54.5 mm to (159.4, 129.3)
- moved REF** 23.2 mm to (208.4, 161.0)
- moved L1 9.22 mm to (137.8, 116.9)
- moved RT1 9.22 mm to (130.4, 124.3)
- moved Q5 9.20 mm to (177.2, 94.9)
- moved Q6 9.20 mm to (192.2, 94.9)
- moved Q13 9.20 mm to (172.2, 227.1)
- moved Q14 9.20 mm to (187.2, 227.1)
- moved L2 9.20 mm to (137.8, 213.6)
- moved REF** 9.20 mm to (160.5, 210.7)
- moved RT4 9.20 mm to (130.4, 198.2)
- moved REF** 9.10 mm to (160.6, 111.3)
- moved REF** 1.80 mm to (172.1, 161.0)
- moved C300 0.28 mm to (153.0, 149.7)
Routing:
- net (no net): track 0.00 -> 113.8 mm
- net Net-(RT2-Pad2): track 136.0 -> 31.2 mm, vias 2 -> 1
- net Net-(RT5-Pad1): track 139.2 -> 45.3 mm
- net /Rsense1: track 109.3 -> 123.2 mm
- net /Rsense2: track 115.8 -> 128.9 mm
- net /LO1: track 203.8 -> 213.1 mm
- net /LO2: track 207.6 -> 216.8 mm
- net Net-(RT1-Pad2): track 39.9 -> 43.7 mm
- net Net-(RT4-Pad1): track 45.2 -> 49.0 mm
- net /12V: track 35.6 -> 35.0 mm
Other:
- board size 170 x 158.2 mm -> 363.3 x 275.3 mm
