File: LM5032 2 Board Design/LM5032 Switching Board Copper Inlay.kicad_sch (KiCad schematic)
At the start: 89 parts, among them Q1 NMOS, Q10 NMOS, Q11 NMOS, Q12 NMOS, Q13 NMOS, Q14 NMOS, Q15 NMOS, Q16 NMOS, Q2 NMOS, Q3 NMOS, Q4 NMOS, Q5 NMOS, Q6 NMOS, Q7 NMOS, Q8 NMOS, Q9 NMOS, U3 UCC27712DR, U4 UCC27712DR

Commit message: update
Parts:
- RT1, RT2, RT3, RT4, RT5, RT6: value 36.5k -> 10k
Changed lines of the file:
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@@
       (effects (font (size 1.27 1.27)))
     )
-    (property "Value" "36.5k" (at 68.58 247.65 90)
+    (property "Value" "10k" (at 68.58 247.65 90)
       (effects (font (size 1.27 1.27)))
     )
@@
       (effects (font (size 1.27 1.27)) hide)
     )
-    (property "Datasheet" "~" (at 68.58 245.11 0)
+    (property "Datasheet" "NTCG163JX103DT1S" (at 68.58 245.11 0)
       (effects (font (size 1.27 1.27)) hide)
     )
@@
       (effects (font (size 1.27 1.27)))
     )
-    (property "Value" "36.5k" (at 68.58 217.17 90)
+    (property "Value" "10k" (at 68.58 217.17 90)
       (effects (font (size 1.27 1.27)))
     )
@@
       (effects (font (size 1.27 1.27)) hide)
     )
-    (property "Datasheet" "~" (at 68.58 214.63 0)
+    (property "Datasheet" "NTCG163JX103DT1S" (at 68.58 214.63 0)
       (effects (font (size 1.27 1.27)) hide)
     )
@@
       (effects (font (size 1.27 1.27)))
     )
-    (property "Value" "36.5k" (at 68.58 227.33 90)
+    (property "Value" "10k" (at 68.58 227.33 90)
       (effects (font (size 1.27 1.27)))
     )
@@
       (effects (font (size 1.27 1.27)) hide)
     )
-    (property "Datasheet" "~" (at 68.58 224.79 0)
+    (property "Datasheet" "NTCG163JX103DT1S" (at 68.58 224.79 0)
       (effects (font (size 1.27 1.27)) hide)
     )
@@
       (effects (font (size 1.27 1.27)))
     )
-    (property "Value" "36.5k" (at 68.58 237.49 90)
+    (property "Value" "10k" (at 68.58 237.49 90)
       (effects (font (size 1.27 1.27)))
     )
@@
       (effects (font (size 1.27 1.27)) hide)
     )
-    (property "Datasheet" "~" (at 68.58 234.95 0)
+    (property "Datasheet" "NTCG163JX103DT1S" (at 68.58 234.95 0)
       (effects (font (size 1.27 1.27)) hide)
     )
@@
       (effects (font (size 1.27 1.27)))
     )
-    (property "Value" "36.5k" (at 68.58 257.81 90)
+    (property "Value" "10k" (at 68.58 257.81 90)
       (effects (font (size 1.27 1.27)))
     )
@@
       (effects (font (size 1.27 1.27)) hide)
     )
-    (property "Datasheet" "~" (at 68.58 255.27 0)
+    (property "Datasheet" "NTCG163JX103DT1S" (at 68.58 255.27 0)
       (effects (font (size 1.27 1.27)) hide)
     )
@@
       (effects (font (size 1.27 1.27)))
     )
-    (property "Value" "36.5k" (at 68.58 207.01 90)
+    (property "Value" "10k" (at 68.58 207.01 90)
       (effects (font (size 1.27 1.27)))
     )
@@
       (effects (font (size 1.27 1.27)) hide)
     )
-    (property "Datasheet" "~" (at 68.58 204.47 0)
-      (effects (font (size 1.27 1.27)) hide)
-    )
+    (property "Datasheet" "NTCG163JX103DT1S" (at 68.58 204.47 0)
+      (effects (font (size 1.27 1.27)) hide)
+    )
